Commit message: added camera plugin

File: axlr_description/urdf/axlr_gazebo.urdf.xacro (robot description, xacro)
@@ -39,3 +39,15 @@
           </plugin>
     </gazebo>
+    <gazebo reference="camera_link">
+        <material>Gazebo/Black</material>
+        <sensor name="camera" type="camera">
+            <pose>0 0 0 0 0 0</pose>
+            <visualize>true</visualize>
+            <update_rate>10.0</update_rate>
+            <plugin name="camera_plugin" filename="libgazebo_ros_camera.so">
+                <!-- <frame_name>camera_link</frame_name> -->
+                <frame_name>camera_link_optical</frame_name> <!-- Frame fix-->
+            </plugin>
+        </sensor>
+    </gazebo>
 </robot>

File: axlr_description/urdf/main.urdf.xacro (robot description, xacro)
@@ -1,6 +1,7 @@
 <?xml version="1.0"?>
 <robot name="my_robot" xmlns:xacro="http://www.ros.org/wiki/xacro">
-    <xacro:include filename="misc_properties.urdf.xacro"/>
-    <xacro:include filename="mobile_base.urdf.xacro"/>
-    <xacro:include filename="mobile_base_gazebo.urdf.xacro"/>
+    <xacro:include filename="axlr_properties.urdf.xacro"/>
+    <xacro:include filename="axlr_base.urdf.xacro"/>
+    <xacro:include filename="axlr_camera.urdf.xacro"/>
+    <xacro:include filename="axlr_gazebo.urdf.xacro"/>
 </robot>

Commit message: added arm

File: axlr_description/urdf/axlr_gazebo.urdf.xacro (robot description, xacro)
@@ -51,3 +51,27 @@
         </sensor>
     </gazebo>
+    <!-- Arm Adaptation for Gazebo-->
+    <gazebo reference= "arm_base_link">
+        <material>Gazebo/Orange</material>
+    </gazebo>
+    <gazebo reference= "fore_arm_link">
+        <material>Gazebo/Yellow</material>
+    </gazebo>
+    <gazebo reference= "hand_link">
+        <material>Gazebo/Orange</material>
+    </gazebo>
+    <gazebo>
+        <plugin name="axlr_arm_state_publisher"
+            filename="libgazebo_ros_joint_state_publisher.so">
+            <update_rate>10</update_rate>
+            <joint_name>arm_base_fore_arm_joint</joint_name>
+            <joint_name>fore_arm_hand_joint</joint_name>
+        </plugin>
+    </gazebo>
+    <gazebo>
+        <plugin name="gazebo_ros_joint_pose_trajectory"
+            filename="libgazebo_ros_joint_pose_trajectory.so">
+            <update_rate>2</update_rate>
+        </plugin>
+    </gazebo>
 </robot>

File: axlr_description/urdf/main.urdf.xacro (robot description, xacro)
@@ -3,5 +3,11 @@
     <xacro:include filename="axlr_properties.urdf.xacro"/>
     <xacro:include filename="axlr_base.urdf.xacro"/>
+    <xacro:include filename="axlr_arm.urdf.xacro"/>
     <xacro:include filename="axlr_camera.urdf.xacro"/>
     <xacro:include filename="axlr_gazebo.urdf.xacro"/>
+    <joint name="base_link_arm_base_joint" type="fixed">
+        <parent link="base_link"/>
+        <child link="arm_base_link"/>
+        <origin xyz="${base_length/4} 0.0 ${base_height}" rpy="0.0 0.0 0.0"/>
+    </joint>
 </robot>

Commit message: added lidar

File: axlr_description/urdf/axlr_gazebo.urdf.xacro (robot description, xacro)
@@ -75,3 +75,32 @@
         </plugin>
     </gazebo>
+    <!-- LIDAR  -->
+    <gazebo reference="lidar_link">
+        <material>Gazebo/Black</material>
+        <sensor name="laser" type="ray">
+            <pose> 0 0 0 0 0 0 </pose>
+            <visualize>false</visualize>
+            <update_rate>10</update_rate>
+            <ray>
+                <scan>
+                    <horizontal>
+                        <samples>360</samples>
+                        <min_angle>-3.14</min_angle>
+                        <max_angle>3.14</max_angle>
+                    </horizontal>
+                </scan>
+                <range>
+                    <min>0.3</min>
+                    <max>12</max>
+                </range>
+            </ray>
+            <plugin name="laser_controller" filename="libgazebo_ros_ray_sensor.so">
+                <ros>
+                    <argument>~/out:=scan</argument>
+                </ros>
+                <output_type>sensor_msgs/LaserScan</output_type>
+                <frame_name>laser_link</frame_name>
+            </plugin>
+        </sensor>
+    </gazebo>
 </robot>

File: axlr_description/urdf/main.urdf.xacro (robot description, xacro)
@@ -3,4 +3,5 @@
     <xacro:include filename="axlr_properties.urdf.xacro"/>
     <xacro:include filename="axlr_base.urdf.xacro"/>
+    <xacro:include filename="axlr_lidar.urdf.xacro"/>
     <xacro:include filename="axlr_arm.urdf.xacro"/>
     <xacro:include filename="axlr_camera.urdf.xacro"/>
